File: Hardware/BackPlane/BackPlane.kicad_pcb (KiCad board)
At the start: 2 copper layers, 117 x 97 mm, 19 parts, among them J101 CAN, J102 i²c, J103 Power Harness, J104 GPIO, U101 COMPUTER, U102 CARD 0, U103 CARD 1, U104 CARD 2, U105 CARD 3

Commit message: Add all
Connections:
- J103 pad 5: Net-(J103-Pin_5) -> +12V
- U101 pad 23: unconnected-(U101-UNUSED1-Pad23) -> /UNUSED1
- U101 pad 24: unconnected-(U101-UNUSED2-Pad24) -> /UNUSED2
- U101 pad 25: unconnected-(U101-UNUSED3-Pad25) -> /UNUSED3
- U101 pad 26: unconnected-(U101-UNUSED4-Pad26) -> /UNUSED4
- U102 pad 23: unconnected-(U102-UNUSED1-Pad23) -> /UNUSED1
- U102 pad 24: unconnected-(U102-UNUSED2-Pad24) -> /UNUSED2
- U102 pad 25: unconnected-(U102-UNUSED3-Pad25) -> /UNUSED3
- U102 pad 26: unconnected-(U102-UNUSED4-Pad26) -> /UNUSED4
- U102 pad 29: unconnected-(U102-UNUSED5-Pad29) -> +5V
- U103 pad 23: unconnected-(U103-UNUSED1-Pad23) -> /UNUSED1
- U103 pad 24: unconnected-(U103-UNUSED2-Pad24) -> /UNUSED2
- U103 pad 25: unconnected-(U103-UNUSED3-Pad25) -> /UNUSED3
- U103 pad 26: unconnected-(U103-UNUSED4-Pad26) -> /UNUSED4
- U103 pad 29: unconnected-(U103-UNUSED5-Pad29) -> +5V
- U104 pad 23: unconnected-(U104-UNUSED1-Pad23) -> /UNUSED1
- U104 pad 24: unconnected-(U104-UNUSED2-Pad24) -> /UNUSED2
- U104 pad 25: unconnected-(U104-UNUSED3-Pad25) -> /UNUSED3
- U104 pad 26: unconnected-(U104-UNUSED4-Pad26) -> /UNUSED4
- U104 pad 29: unconnected-(U104-UNUSED5-Pad29) -> +5V
- U105 pad 23: unconnected-(U105-UNUSED1-Pad23) -> /UNUSED1
- U105 pad 24: unconnected-(U105-UNUSED2-Pad24) -> /UNUSED2
- U105 pad 25: unconnected-(U105-UNUSED3-Pad25) -> /UNUSED3
- U105 pad 26: unconnected-(U105-UNUSED4-Pad26) -> /UNUSED4
- U105 pad 29: unconnected-(U105-UNUSED5-Pad29) -> +5V
Routing:
- net /UNUSED4: track 0.00 -> 91.4 mm
- net /UNUSED1: track 0.00 -> 91.0 mm
- net +5V: track 44.4 -> 135.2 mm
- net /UNUSED3: track 0.00 -> 90.9 mm
- net /UNUSED2: track 0.00 -> 90.8 mm
- net unconnected-(U101-UNUSED4-Pad26): track 0.65 -> 0.00 mm
