File: Hardware/FennecModem/radio.kicad_sch (KiCad schematic)
At the start: 15 parts, among them J201 Conn_Coaxial, U201 DRA818V

Commit message: Route!
Parts:
- added TP1: SleepTP, TestPoint:TestPoint_Bridge_Pitch2.0mm_Drill0.7mm, symbol Connector:TestPoint_Small
- added TP2: H/L, TestPoint:TestPoint_Bridge_Pitch2.0mm_Drill0.7mm, symbol Connector:TestPoint_Small
- added TP3: PTT, TestPoint:TestPoint_Bridge_Pitch2.0mm_Drill0.7mm, symbol Connector:TestPoint_Small
- added TP4: AudioOut, TestPoint:TestPoint_Bridge_Pitch2.0mm_Drill0.7mm, symbol Connector:TestPoint_Small
- added TP5: AudioIn, TestPoint:TestPoint_Bridge_Pitch2.0mm_Drill0.7mm, symbol Connector:TestPoint_Small
- added TP6: SQL, TestPoint:TestPoint_Bridge_Pitch2.0mm_Drill0.7mm, symbol Connector:TestPoint_Small
- added TP7: TXD, TestPoint:TestPoint_Bridge_Pitch2.0mm_Drill0.7mm, symbol Connector:TestPoint_Small
- added TP8: RXD, TestPoint:TestPoint_Bridge_Pitch2.0mm_Drill0.7mm, symbol Connector:TestPoint_Small
Connections:
- net +5V: no longer R201.2, R202.2, R203.2, R204.2, R205.2
- net AudioIn: now also TP5.1
- net AudioOut: now also TP4.1
- net H/L: now also TP2.1
- net RXD: now also TP8.1
- net SQL: now also TP6.1
- net Sleep: now also TP1.1
- net TXD: now also TP7.1
- net at R206.2, U201.5 (PTT): now also TP3.1
- new net +3.3V: R201.2, R202.2, R203.2, R204.2, R205.2
Other:
- moved on the sheet: D202, D203, D204, R201, R203, R204, R205, R206
